Commit message: bug fix

File: wheels.xacro (robot description, xacro)
@@ -27,5 +27,5 @@
     <joint name="back_left_wheel_joint" type="continuous">
       <parent link="base_link"/>
-      <child link="${back_left_wheel}"/>
+      <child link="back_left_wheel"/>
       <origin xyz="${x} ${y} ${z}"/>
       <axis xyz="0 1 0"/>
@@ -53,5 +53,5 @@
     <joint name="back_right_wheel_joint" type="continuous">
       <parent link="base_link"/>
-      <child link="${back_left_wheel}"/>
+      <child link="back_right_wheel"/>
       <origin xyz="${x} ${y} ${z}"/>
       <axis xyz="0 1 0"/>
@@ -79,5 +79,5 @@
     <joint name="front_left_wheel_joint" type="continuous">
       <parent link="base_link"/>
-      <child link="${back_left_wheel}"/>
+      <child link="front_left_wheel"/>
       <origin xyz="${x} ${y} ${z}"/>
       <axis xyz="0 1 0"/>
@@ -105,5 +105,5 @@
     <joint name="front_right_wheel_joint" type="continuous">
       <parent link="base_link"/>
-      <child link="${back_left_wheel}"/>
+      <child link="front_right_wheel"/>
       <origin xyz="${x} ${y} ${z}"/>
       <axis xyz="0 1 0"/>

Commit message: bug fixes

File: wheels.xacro (robot description, xacro)
@@ -5,4 +5,16 @@
     <xacro:property name="wheel_mass" value="0.1"/>
     <xacro:property name="wheel_inertia" value="0.001 0.0 0.0 0.001 0.0 0.001"/>
+    <xacro:property name="blx" value="-0.2"/>
+    <xacro:property name="bly" value="-0.125"/>
+    <xacro:property name="blz" value="0"/>
+    <xacro:property name="brx" value="-0.2"/>
+    <xacro:property name="bry" value="0.125"/>
+    <xacro:property name="brz" value="0"/>
+    <xacro:property name="flx" value="0"/>
+    <xacro:property name="fly" value="-0.125"/>
+    <xacro:property name="flz" value="0"/>
+    <xacro:property name="frx" value="0"/>
+    <xacro:property name="fry" value="-0.125"/>
+    <xacro:property name="frz" value="0"/>
     <link name="back_left_wheel">
       <visual>
@@ -28,5 +40,5 @@
       <parent link="base_link"/>
       <child link="back_left_wheel"/>
-      <origin xyz="${x} ${y} ${z}"/>
+      <origin xyz="${blx} ${bly} ${blz}"/>
       <axis xyz="0 1 0"/>
     </joint>
@@ -54,5 +66,5 @@
       <parent link="base_link"/>
       <child link="back_right_wheel"/>
-      <origin xyz="${x} ${y} ${z}"/>
+      <origin xyz="${brx} ${bry} ${brz}"/>
       <axis xyz="0 1 0"/>
     </joint>
@@ -78,7 +90,7 @@
     </link>
     <joint name="front_left_wheel_joint" type="continuous">
-      <parent link="base_link"/>
+      <parent link="front_wheel_steering_link"/>
       <child link="front_left_wheel"/>
-      <origin xyz="${x} ${y} ${z}"/>
+      <origin xyz="${flx} ${fly} ${flz}"/>
       <axis xyz="0 1 0"/>
     </joint>
@@ -104,7 +116,7 @@
     </link>
     <joint name="front_right_wheel_joint" type="continuous">
-      <parent link="base_link"/>
+      <parent link="front_wheel_steering_link"/>
       <child link="front_right_wheel"/>
-      <origin xyz="${x} ${y} ${z}"/>
+      <origin xyz="${frx} ${fry} ${frz}"/>
       <axis xyz="0 1 0"/>
     </joint>

Commit message: tire size

File: wheels.xacro (robot description, xacro)
@@ -1,5 +1,5 @@
 <?xml version="1.0"?>
 <robot xmlns:xacro="http://www.ros.org/wiki/xacro">
-    <xacro:property name="wheel_radius" value="0.05"/>
+    <xacro:property name="wheel_radius" value="0.075"/>
     <xacro:property name="wheel_length" value="0.05"/>
     <xacro:property name="wheel_mass" value="0.1"/>
