Commit message: xmlns issue

File: base_link.xacro (robot description, xacro)
@@ -1,3 +1,4 @@
 <?xml version="1.0"?>
+<robot xmlns:xacro="http://www.ros.org/wiki/xacro">
 <xacro:macro name="base_link_macro">
   <xacro:property name="base_size" value="0.4 0.2 0.1"/>

File: steering_mechanism.xacro (robot description, xacro)
@@ -1,3 +1,4 @@
 <?xml version="1.0"?>
+<robot xmlns:xacro="http://www.ros.org/wiki/xacro">
 <xacro:macro name="steering_mechanism_macro">
   <xacro:property name="sphere_radius" value="0.025"/>
@@ -71,2 +72,3 @@
     <origin xyz="0 0.125 0"/>
     <axis xyz="0 1 0"/>
+  </joint>

File: wheels.xacro (robot description, xacro)
@@ -1,3 +1,4 @@
 <?xml version="1.0"?>
+<robot xmlns:xacro="http://www.ros.org/wiki/xacro">
 <xacro:macro name="wheel_macro" params="name x y z">
   <xacro:property name="wheel_radius" value="0.075"/>

Commit message: better structure

File: base_link.xacro (robot description, xacro)
@@ -1,26 +1,27 @@
 <?xml version="1.0"?>
 <robot xmlns:xacro="http://www.ros.org/wiki/xacro">
-<xacro:macro name="base_link_macro">
-  <xacro:property name="base_size" value="0.4 0.2 0.1"/>
-  <xacro:property name="base_mass" value="1.0"/>
-  <xacro:property name="base_inertia" value="0.01 0.0 0.0 0.01 0.0 0.01"/>
-  <link name="base_link">
-    <visual>
-      <geometry>
-        <box size="${base_size}"/> <!-- Dimensions of the base -->
-      </geometry>
-      <material name="gray"/>
-    </visual>
-    <collision>
-      <geometry>
-        <box size="${base_size}"/>
-      </geometry>
-    </collision>
-    <inertial>
-      <mass value="${base_mass}"/>
-      <inertia ixx="${base_inertia.split(' ')[0]}" ixy="${base_inertia.split(' ')[1]}" ixz="${base_inertia.split(' ')[2]}"
-              iyy="${base_inertia.split(' ')[3]}" iyz="${base_inertia.split(' ')[4]}" izz="${base_inertia.split(' ')[5]}"/>
-    </inertial>
-  </link>
-</xacro:macro>
-<base_link_macro/>
+  <xacro:macro name="base_link">
+    <xacro:property name="base_size" value="0.4 0.2 0.1"/>
+    <xacro:property name="base_mass" value="1.0"/>
+    <xacro:property name="base_inertia" value="0.01 0.0 0.0 0.01 0.0 0.01"/>
+    <link name="base_link">
+      <visual>
+        <geometry>
+          <box size="${base_size}"/> <!-- Dimensions of the base -->
+        </geometry>
+        <material name="gray"/>
+      </visual>
+      <collision>
+        <geometry>
+          <box size="${base_size}"/>
+        </geometry>
+      </collision>
+      <inertial>
+        <mass value="${base_mass}"/>
+        <inertia ixx="${base_inertia.split(' ')[0]}" ixy="${base_inertia.split(' ')[1]}" ixz="${base_inertia.split(' ')[2]}"
+                iyy="${base_inertia.split(' ')[3]}" iyz="${base_inertia.split(' ')[4]}" izz="${base_inertia.split(' ')[5]}"/>
+      </inertial>
+    </link>
+  </xacro:macro>
+  <base_link/>
+</robot>

File: primeberry1.urdf.xacro (robot description, xacro)
@@ -6,5 +6,5 @@
   <xacro:include filename="steering_mechanism.xacro"/>
   <xacro:property name="pi" value="3.14159265359"/>
-  <link name="world"></link>
+  <link name="world"/>
   <joint name="base_joint" type="fixed">
     <origin xyz="1.5 1.0 0.0" rpy="0.0 0.0 0.0"/>

File: steering_mechanism.xacro (robot description, xacro)
@@ -1,74 +1,77 @@
 <?xml version="1.0"?>
 <robot xmlns:xacro="http://www.ros.org/wiki/xacro">
-<xacro:macro name="steering_mechanism_macro">
-  <xacro:property name="sphere_radius" value="0.025"/>
-  <xacro:property name="sphere_mass" value="0.05"/>
-  <xacro:property name="sphere_inertia" value="0.0001 0.0 0.0 0.0001 0.0 0.0001"/>
-  <xacro:property name="steering_size" value="0.1 0.2 0.05"/>
-  <xacro:property name="steering_mass" value="0.2"/>
-  <xacro:property name="steering_inertia" value="0.002 0.0 0.0 0.002 0.0 0.002"/>
-  <!-- Link for the sphere -->
-  <link name="steering_sphere">
-    <visual>
-      <geometry>
-        <sphere radius="${sphere_radius}"/>
-      </geometry>
-      <material name="blue"/>
-    </visual>
-    <collision>
-      <geometry>
-        <sphere radius="${sphere_radius}"/>
-      </geometry>
-    </collision>
-    <inertial>
-      <mass value="${sphere_mass}"/>
-      <inertia ixx="${sphere_inertia.split(' ')[0]}" ixy="${sphere_inertia.split(' ')[1]}" ixz="${sphere_inertia.split(' ')[2]}"
-              iyy="${sphere_inertia.split(' ')[3]}" iyz="${sphere_inertia.split(' ')[4]}" izz="${sphere_inertia.split(' ')[5]}"/>
-    </inertial>
-  </link>
-  <!-- Joint connecting the sphere to the base link -->
-  <joint name="sphere_to_base_joint" type="fixed">
-    <parent link="base_link"/>
-    <child link="steering_sphere"/>
-    <origin xyz="0.225 0 0"/>
-  </joint>
-  <!-- Joint connecting the sphere to the steering mechanism -->
-  <joint name="sphere_to_steering_joint" type="revolute">
-    <parent link="steering_sphere"/>
-    <child link="front_wheel_steering_link"/>
-    <origin xyz="0.075 0 0"/> <!-- Position the sphere below the steering mechanism -->
-    <axis xyz="0 0 1"/> <!-- Define the axis of rotation -->
-    <limit lower="-0.75" upper="0.75" effort="1.0" velocity="1.0"/> <!-- Define the limits, effort, and velocity -->
-  </joint>
-  <!-- Link for the steering mechanism -->
-  <link name="front_wheel_steering_link">
-    <visual>
-      <geometry>
-        <box size="${steering_size}"/>
-      </geometry>
-      <material name="gray"/>
-    </visual>
-    <collision>
-      <geometry>
-        <box size="${steering_size}"/>
-      </geometry>
-    </collision>
-    <inertial>
-      <mass value="${steering_mass}"/>
-      <inertia ixx="${steering_inertia.split(' ')[0]}" ixy="${steering_inertia.split(' ')[1]}" ixz="${steering_inertia.split(' ')[2]}"
-              iyy="${steering_inertia.split(' ')[3]}" iyz="${steering_inertia.split(' ')[4]}" izz="${steering_inertia.split(' ')[5]}"/>
-    </inertial>
-  </link>
-  <!-- Joints for the front wheels attached to the steering mechanism -->
-  <joint name="front_left_wheel_steering_joint" type="continuous">
-    <parent link="front_wheel_steering_link"/>
-    <child link="front_left_wheel"/>
-    <origin xyz="0 -0.125 0"/>
-    <axis xyz="0 1 0"/>
-  </joint>
-  <joint name="front_right_wheel_steering_joint" type="continuous">
-    <parent link="front_wheel_steering_link"/>
-    <child link="front_right_wheel"/>
-    <origin xyz="0 0.125 0"/>
-    <axis xyz="0 1 0"/>
-  </joint>
+  <xacro:macro name="steering_mechanism_macro">
+    <xacro:property name="sphere_radius" value="0.025"/>
+    <xacro:property name="sphere_mass" value="0.05"/>
+    <xacro:property name="sphere_inertia" value="0.0001 0.0 0.0 0.0001 0.0 0.0001"/>
+    <xacro:property name="steering_size" value="0.1 0.2 0.05"/>
+    <xacro:property name="steering_mass" value="0.2"/>
+    <xacro:property name="steering_inertia" value="0.002 0.0 0.0 0.002 0.0 0.002"/>
+    <!-- Link for the sphere -->
+    <link name="steering_sphere">
+      <visual>
+        <geometry>
+          <sphere radius="${sphere_radius}"/>
+        </geometry>
+        <material name="blue"/>
+      </visual>
+      <collision>
+        <geometry>
+          <sphere radius="${sphere_radius}"/>
+        </geometry>
+      </collision>
+      <inertial>
+        <mass value="${sphere_mass}"/>
+        <inertia ixx="${sphere_inertia.split(' ')[0]}" ixy="${sphere_inertia.split(' ')[1]}" ixz="${sphere_inertia.split(' ')[2]}"
+                iyy="${sphere_inertia.split(' ')[3]}" iyz="${sphere_inertia.split(' ')[4]}" izz="${sphere_inertia.split(' ')[5]}"/>
+      </inertial>
+    </link>
+    <!-- Joint connecting the sphere to the base link -->
+    <joint name="sphere_to_base_joint" type="fixed">
+      <parent link="base_link"/>
+      <child link="steering_sphere"/>
+      <origin xyz="0.225 0 0"/>
+    </joint>
+    <!-- Joint connecting the sphere to the steering mechanism -->
+    <joint name="sphere_to_steering_joint" type="revolute">
+      <parent link="steering_sphere"/>
+      <child link="front_wheel_steering_link"/>
+      <origin xyz="0.075 0 0"/> <!-- Position the sphere below the steering mechanism -->
+      <axis xyz="0 0 1"/> <!-- Define the axis of rotation -->
+      <limit lower="-0.75" upper="0.75" effort="1.0" velocity="1.0"/> <!-- Define the limits, effort, and velocity -->
+    </joint>
+    <!-- Link for the steering mechanism -->
+    <link name="front_wheel_steering_link">
+      <visual>
+        <geometry>
+          <box size="${steering_size}"/>
+        </geometry>
+        <material name="gray"/>
+      </visual>
+      <collision>
+        <geometry>
+          <box size="${steering_size}"/>
+        </geometry>
+      </collision>
+      <inertial>
+        <mass value="${steering_mass}"/>
+        <inertia ixx="${steering_inertia.split(' ')[0]}" ixy="${steering_inertia.split(' ')[1]}" ixz="${steering_inertia.split(' ')[2]}"
+                iyy="${steering_inertia.split(' ')[3]}" iyz="${steering_inertia.split(' ')[4]}" izz="${steering_inertia.split(' ')[5]}"/>
+      </inertial>
+    </link>
+    <!-- Joints for the front wheels attached to the steering mechanism -->
+    <joint name="front_left_wheel_steering_joint" type="continuous">
+      <parent link="front_wheel_steering_link"/>
+      <child link="front_left_wheel"/>
+      <origin xyz="0 -0.125 0"/>
+      <axis xyz="0 1 0"/>
+    </joint>
+    <joint name="front_right_wheel_steering_joint" type="continuous">
+      <parent link="front_wheel_steering_link"/>
+      <child link="front_right_wheel"/>
+      <origin xyz="0 0.125 0"/>
+      <axis xyz="0 1 0"/>
+    </joint>
+  </xacro:macro>
+  <steering_mechanism_macro/>
+</robot>

File: wheels.xacro (robot description, xacro)
@@ -1,38 +1,39 @@
 <?xml version="1.0"?>
 <robot xmlns:xacro="http://www.ros.org/wiki/xacro">
-<xacro:macro name="wheel_macro" params="name x y z">
-  <xacro:property name="wheel_radius" value="0.075"/>
-  <xacro:property name="wheel_length" value="0.05"/>
-  <xacro:property name="wheel_mass" value="0.1"/>
-  <xacro:property name="wheel_inertia" value="0.001 0.0 0.0 0.001 0.0 0.001"/>
-  <link name="${name}">
-    <visual>
-      <origin rpy="0.0 ${pi/2} ${pi/2}"/>
-      <geometry>
-        <cylinder length="${wheel_length}" radius="${wheel_radius}"/>
-      </geometry>
-      <material name="black"/>
-    </visual>
-    <collision>
-      <origin rpy="0.0 ${pi/2} ${pi/2}"/>
-      <geometry>
-        <cylinder length="${wheel_length}" radius="${wheel_radius}"/>
-      </geometry>
-    </collision>
-    <inertial>
-      <mass value="${wheel_mass}"/>
-      <inertia ixx="${wheel_inertia.split(' ')[0]}" ixy="${wheel_inertia.split(' ')[1]}" ixz="${wheel_inertia.split(' ')[2]}"
-              iyy="${wheel_inertia.split(' ')[3]}" iyz="${wheel_inertia.split(' ')[4]}" izz="${wheel_inertia.split(' ')[5]}"/>
-    </inertial>
-  </link>
-  <joint name="${name}_joint" type="continuous">
-    <parent link="base_link"/>
-    <child link="${name}"/>
-    <origin xyz="${x} ${y} ${z}"/>
-    <axis xyz="0 1 0"/>
-  </joint>
-</xacro:macro>
-<wheel_macro name="back_left_wheel" x="-0.2" y="-0.125" z="0"/>
-<wheel_macro name="back_right_wheel" x="-0.2" y="0.125" z="0"/>
-<wheel_macro name="front_left_wheel" x="0.2" y="-0.125" z="0"/>
-<wheel_macro name="front_right_wheel" x="0.2" y="0.125" z="0"/>
+  <xacro:macro name="wheel_macro" params="name x y z">
+    <xacro:property name="wheel_radius" value="0.05"/>
+    <xacro:property name="wheel_length" value="0.05"/>
+    <xacro:property name="wheel_mass" value="0.1"/>
+    <xacro:property name="wheel_inertia" value="0.001 0.0 0.0 0.001 0.0 0.001"/>
+    <link name="${name}">
+      <visual>
+        <origin rpy="0.0 ${pi/2} ${pi/2}"/>
+        <geometry>
+          <cylinder length="${wheel_length}" radius="${wheel_radius}"/>
+        </geometry>
+        <material name="black"/>
+      </visual>
+      <collision>
+        <origin rpy="0.0 ${pi/2} ${pi/2}"/>
+        <geometry>
+          <cylinder length="${wheel_length}" radius="${wheel_radius}"/>
+        </geometry>
+      </collision>
+      <inertial>
+        <mass value="${wheel_mass}"/>
+        <inertia ixx="${wheel_inertia.split(' ')[0]}" ixy="${wheel_inertia.split(' ')[1]}" ixz="${wheel_inertia.split(' ')[2]}"
+                iyy="${wheel_inertia.split(' ')[3]}" iyz="${wheel_inertia.split(' ')[4]}" izz="${wheel_inertia.split(' ')[5]}"/>
+      </inertial>
+    </link>
+    <joint name="${name}_joint" type="continuous">
+      <parent link="base_link"/>
+      <child link="${name}"/>
+      <origin xyz="${x} ${y} ${z}"/>
+      <axis xyz="0 1 0"/>
+    </joint>
+  </xacro:macro>
+  <wheel_macro name="back_left_wheel" x="-0.2" y="-0.125" z="0"/>
+  <wheel_macro name="back_right_wheel" x="-0.2" y="0.125" z="0"/>
+  <wheel_macro name="front_left_wheel" x="0.2" y="-0.125" z="0"/>
+  <wheel_macro name="front_right_wheel" x="0.2" y="0.125" z="0"/>
+</robot>

Commit message: removed macro

File: base_link.xacro (robot description, xacro)
@@ -1,5 +1,4 @@
 <?xml version="1.0"?>
 <robot xmlns:xacro="http://www.ros.org/wiki/xacro">
-  <xacro:macro name="base_link">
     <xacro:property name="base_size" value="0.4 0.2 0.1"/>
     <xacro:property name="base_mass" value="1.0"/>
@@ -23,5 +22,3 @@
       </inertial>
     </link>
-  </xacro:macro>
-  <base_link/>
 </robot>

File: steering_mechanism.xacro (robot description, xacro)
@@ -1,5 +1,4 @@
 <?xml version="1.0"?>
 <robot xmlns:xacro="http://www.ros.org/wiki/xacro">
-  <xacro:macro name="steering_mechanism_macro">
     <xacro:property name="sphere_radius" value="0.025"/>
     <xacro:property name="sphere_mass" value="0.05"/>
@@ -73,5 +72,3 @@
       <axis xyz="0 1 0"/>
     </joint>
-  </xacro:macro>
-  <steering_mechanism_macro/>
 </robot>

File: wheels.xacro (robot description, xacro)
@@ -1,10 +1,9 @@
 <?xml version="1.0"?>
 <robot xmlns:xacro="http://www.ros.org/wiki/xacro">
-  <xacro:macro name="wheel_macro" params="name x y z">
     <xacro:property name="wheel_radius" value="0.05"/>
     <xacro:property name="wheel_length" value="0.05"/>
     <xacro:property name="wheel_mass" value="0.1"/>
     <xacro:property name="wheel_inertia" value="0.001 0.0 0.0 0.001 0.0 0.001"/>
-    <link name="${name}">
+    <link name="back_left_wheel">
       <visual>
         <origin rpy="0.0 ${pi/2} ${pi/2}"/>
@@ -26,14 +25,87 @@
       </inertial>
     </link>
-    <joint name="${name}_joint" type="continuous">
+    <joint name="back_left_wheel_joint" type="continuous">
       <parent link="base_link"/>
-      <child link="${name}"/>
+      <child link="${back_left_wheel}"/>
       <origin xyz="${x} ${y} ${z}"/>
       <axis xyz="0 1 0"/>
     </joint>
-  </xacro:macro>
-  <wheel_macro name="back_left_wheel" x="-0.2" y="-0.125" z="0"/>
-  <wheel_macro name="back_right_wheel" x="-0.2" y="0.125" z="0"/>
-  <wheel_macro name="front_left_wheel" x="0.2" y="-0.125" z="0"/>
-  <wheel_macro name="front_right_wheel" x="0.2" y="0.125" z="0"/>
+    <link name="back_right_wheel">
+      <visual>
+        <origin rpy="0.0 ${pi/2} ${pi/2}"/>
+        <geometry>
+          <cylinder length="${wheel_length}" radius="${wheel_radius}"/>
+        </geometry>
+        <material name="black"/>
+      </visual>
+      <collision>
+        <origin rpy="0.0 ${pi/2} ${pi/2}"/>
+        <geometry>
+          <cylinder length="${wheel_length}" radius="${wheel_radius}"/>
+        </geometry>
+      </collision>
+      <inertial>
+        <mass value="${wheel_mass}"/>
+        <inertia ixx="${wheel_inertia.split(' ')[0]}" ixy="${wheel_inertia.split(' ')[1]}" ixz="${wheel_inertia.split(' ')[2]}"
+                iyy="${wheel_inertia.split(' ')[3]}" iyz="${wheel_inertia.split(' ')[4]}" izz="${wheel_inertia.split(' ')[5]}"/>
+      </inertial>
+    </link>
+    <joint name="back_right_wheel_joint" type="continuous">
+      <parent link="base_link"/>
+      <child link="${back_left_wheel}"/>
+      <origin xyz="${x} ${y} ${z}"/>
+      <axis xyz="0 1 0"/>
+    </joint>
+<link name="front_left_wheel">
+      <visual>
+        <origin rpy="0.0 ${pi/2} ${pi/2}"/>
+        <geometry>
+          <cylinder length="${wheel_length}" radius="${wheel_radius}"/>
+        </geometry>
+        <material name="black"/>
+      </visual>
+      <collision>
+        <origin rpy="0.0 ${pi/2} ${pi/2}"/>
+        <geometry>
+          <cylinder length="${wheel_length}" radius="${wheel_radius}"/>
+        </geometry>
+      </collision>
+      <inertial>
+        <mass value="${wheel_mass}"/>
+        <inertia ixx="${wheel_inertia.split(' ')[0]}" ixy="${wheel_inertia.split(' ')[1]}" ixz="${wheel_inertia.split(' ')[2]}"
+                iyy="${wheel_inertia.split(' ')[3]}" iyz="${wheel_inertia.split(' ')[4]}" izz="${wheel_inertia.split(' ')[5]}"/>
+      </inertial>
+    </link>
+    <joint name="front_left_wheel_joint" type="continuous">
+      <parent link="base_link"/>
+      <child link="${back_left_wheel}"/>
+      <origin xyz="${x} ${y} ${z}"/>
+      <axis xyz="0 1 0"/>
+    </joint>
+<link name="front_right_wheel">
+      <visual>
+        <origin rpy="0.0 ${pi/2} ${pi/2}"/>
+        <geometry>
+          <cylinder length="${wheel_length}" radius="${wheel_radius}"/>
+        </geometry>
+        <material name="black"/>
+      </visual>
+      <collision>
+        <origin rpy="0.0 ${pi/2} ${pi/2}"/>
+        <geometry>
+          <cylinder length="${wheel_length}" radius="${wheel_radius}"/>
+        </geometry>
+      </collision>
+      <inertial>
+        <mass value="${wheel_mass}"/>
+        <inertia ixx="${wheel_inertia.split(' ')[0]}" ixy="${wheel_inertia.split(' ')[1]}" ixz="${wheel_inertia.split(' ')[2]}"
+                iyy="${wheel_inertia.split(' ')[3]}" iyz="${wheel_inertia.split(' ')[4]}" izz="${wheel_inertia.split(' ')[5]}"/>
+      </inertial>
+    </link>
+    <joint name="front_right_wheel_joint" type="continuous">
+      <parent link="base_link"/>
+      <child link="${back_left_wheel}"/>
+      <origin xyz="${x} ${y} ${z}"/>
+      <axis xyz="0 1 0"/>
+    </joint>
 </robot>

Commit message: some changes

File: base_link.xacro (robot description, xacro)
@@ -22,3 +22,6 @@
       </inertial>
     </link>
+      <gazebo reference="base_link">
+    <material>Gazebo/Gray</material>
+  </gazebo>
 </robot>

File: steering_mechanism.xacro (robot description, xacro)
@@ -26,4 +26,7 @@
       </inertial>
     </link>
+    <gazebo reference="steering_sphere">
+      <material>Gazebo/Blue</material>
+    </gazebo>
     <!-- Joint connecting the sphere to the base link -->
     <joint name="sphere_to_base_joint" type="fixed">
@@ -59,4 +62,7 @@
       </inertial>
     </link>
+     <gazebo reference="front_wheel_steering_link">
+    <material>Gazebo/Gray</material>
+    </gazebo>
     <!-- Joints for the front wheels attached to the steering mechanism -->
     <joint name="front_left_wheel_steering_joint" type="continuous">

File: wheels.xacro (robot description, xacro)
@@ -37,4 +37,7 @@
       </inertial>
     </link>
+     <gazebo reference="back_left_wheel">
+    <material>Gazebo/Black</material>
+  </gazebo>
     <joint name="back_left_wheel_joint" type="continuous">
       <parent link="base_link"/>
@@ -63,4 +66,7 @@
       </inertial>
     </link>
+     <gazebo reference="back_right_wheel">
+    <material>Gazebo/Black</material>
+  </gazebo>
     <joint name="back_right_wheel_joint" type="continuous">
       <parent link="base_link"/>
@@ -69,5 +75,5 @@
       <axis xyz="0 1 0"/>
     </joint>
-<link name="front_left_wheel">
+  <link name="front_left_wheel">
       <visual>
         <origin rpy="0.0 ${pi/2} ${pi/2}"/>
@@ -89,4 +95,7 @@
       </inertial>
     </link>
+     <gazebo reference="front_left_wheel">
+    <material>Gazebo/Black</material>
+  </gazebo>
     <joint name="front_left_wheel_joint" type="continuous">
       <parent link="front_wheel_steering_link"/>
@@ -115,4 +124,7 @@
       </inertial>
     </link>
+     <gazebo reference="front_right_wheel">
+    <material>Gazebo/Black</material>
+  </gazebo>
     <joint name="front_right_wheel_joint" type="continuous">
       <parent link="front_wheel_steering_link"/>
